File: Eagle/TG-Final/nivel0.sch (EAGLE design)
At the start: 12 parts

Commit message: Routing placa Actuadores
Parts:
- removed X2: (no value), con-wago-508:W237-02P
- added MOTOR2: (no value), con-wago-508:W237-02P
- BAT001, BAT002, BAT003: value (none) -> 11.1v
- JP1, JP2, JP3, JP4, MOTOR1: value (none) -> (none)
- U$12: value CONECTOR_AUDIO -> CONECTOR_AUDIO2; device aasanchez:CONECTOR_AUDIO -> aasanchez:CONECTOR_AUDIO2
- renumbered X1 to MOTOR1
Connections:
- new net +12V: U$1.PIN18, U$12.ROJO
- new net +24V: U$1.PIN17, U$11.ROJO1
- new net +3V3: U$1.PIN21
- new net +5V: U$1.PIN20
- new net M1-BLACK: MOTOR1-1.KL, U$1.PIN28
- new net M1-RED: MOTOR1-2.KL, U$1.PIN29
- new net M2-BLACK: MOTOR2-1.KL, U$1.PIN31
- new net M2-RED: MOTOR2-2.KL, U$1.PIN30
- new net N$1: U$11.NEGRO1, U$11.ROJO2
- net SERVO01: now also U$1.PIN24
- net SERVO02: now also U$1.PIN27
- net SERVO03: now also U$1.PIN26
- net SERVO04: now also U$1.PIN25
- net VSS: now also U$1.PIN16, U$11.NEGRO2, U$12.NEGRO

Commit message: Routing placa Actuadores. Listo??
Connections:
- removed net +6V: JP1.2, JP2.2, JP3.2, JP4.2
- new net P$1: JP1.2, JP2.2, JP3.2, JP4.2, U$1.PIN19
- new net SENSE1: BAT001.1, U$1.PIN15
- new net SENSE2: BAT002.4, U$1.PIN13
- new net SENSE3: BAT003.1, U$1.PIN14
- net VSS: now also BAT001.4, BAT002.1, BAT003.4
Other:
- note added: "+6V"
- moved on the sheet: BAT001, BAT003
Changed lines of the file:
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@@
 <setting verticaltext="up"/>
 </settings>
-<grid distance="0.1" unitdist="inch" unit="inch" style="lines" multiple="1" display="no" altdistance="0.01" altunitdist="inch" altunit="inch"/>
+<grid distance="0.05" unitdist="inch" unit="inch" style="lines" multiple="1" display="no" altdistance="0.01" altunitdist="inch" altunit="inch"/>
 <layers>
 <layer number="1" name="Top" color="4" fill="1" visible="no" active="no"/>
@@
 <part name="VSS3" library="supply1" deviceset="VSS" device=""/>
 <part name="VSS4" library="supply1" deviceset="VSS" device=""/>
-<part name="SUPPLY1" library="supply2" deviceset="+7V" device="" value="+6V"/>
-<part name="SUPPLY2" library="supply2" deviceset="+7V" device="" value="+6V"/>
-<part name="SUPPLY3" library="supply2" deviceset="+7V" device="" value="+6V"/>
-<part name="SUPPLY4" library="supply2" deviceset="+7V" device="" value="+6V"/>
 <part name="MOTOR1" library="con-wago-508" deviceset="W237-02P" device="" value=" "/>
 <part name="MOTOR2" library="con-wago-508" deviceset="W237-02P" device="" value=" "/>
@@
 <part name="P+5" library="supply1" deviceset="+5V" device=""/>
 <part name="+3V1" library="supply1" deviceset="+3V3" device=""/>
-<part name="+3V2" library="supply1" deviceset="+3V3" device=""/>
+<part name="U$13" library="aasanchez" deviceset="+6V" device=""/>
+<part name="U$14" library="aasanchez" deviceset="+6V" device=""/>
+<part name="U$15" library="aasanchez" deviceset="+6V" device=""/>
+<part name="U$16" library="aasanchez" deviceset="+6V" device=""/>
+<part name="U$17" library="aasanchez" deviceset="+6V" device=""/>
+<part name="VSS8" library="supply1" deviceset="VSS" device=""/>
 </parts>
 <sheets>
@@
 <description>Base</description>
 <plain>
+<text x="100.33" y="27.94" size="1.778" layer="96" rot="R90">+6V</text>
 </plain>
 <instances>
@@
 <instance part="P+5" gate="1" x="104.14" y="27.94" rot="R180"/>
 <instance part="+3V1" gate="G$1" x="111.76" y="27.94" rot="R180"/>
-<instance part="+3V2" gate="G$1" x="96.52" y="27.94" rot="R180"/>
+<instance part="U$13" gate="G$1" x="96.52" y="30.48" rot="R180"/>
 </instances>
 <busses>
@@
 <wire x1="73.66" y1="63.5" x2="78.74" y2="63.5" width="0.1524" layer="91"/>
 <label x="78.74" y="63.5" size="1.778" layer="95"/>
+</segment>
+</net>
+<net name="P$1" class="0">
+<segment>
+<pinref part="U$1" gate="G$1" pin="PIN19"/>
+<pinref part="U$13" gate="G$1" pin="P$1"/>
+<wire x1="73.66" y1="43.18" x2="96.52" y2="43.18" width="0.1524" layer="91"/>
+<wire x1="96.52" y1="43.18" x2="96.52" y2="30.48" width="0.1524" layer="91"/>
+</segment>
+</net>
+<net name="SENSE1" class="0">
+<segment>
+<pinref part="U$1" gate="G$1" pin="PIN15"/>
+<wire x1="43.18" y1="35.56" x2="38.1" y2="35.56" width="0.1524" layer="91"/>
+<label x="27.94" y="35.56" size="1.778" layer="95"/>
+</segment>
+</net>
+<net name="SENSE3" class="0">
+<segment>
+<pinref part="U$1" gate="G$1" pin="PIN14"/>
+<wire x1="43.18" y1="38.1" x2="38.1" y2="38.1" width="0.1524" layer="91"/>
+<label x="27.94" y="38.1" size="1.778" layer="95"/>
+</segment>
+</net>
+<net name="SENSE2" class="0">
+<segment>
+<pinref part="U$1" gate="G$1" pin="PIN13"/>
+<wire x1="43.18" y1="40.64" x2="38.1" y2="40.64" width="0.1524" layer="91"/>
+<label x="27.94" y="40.64" size="1.778" layer="95"/>
 </segment>
 </net>
@@
 </plain>
 <instances>
-<instance part="BAT001" gate="G$1" x="5.08" y="5.08"/>
-<instance part="BAT003" gate="G$1" x="40.64" y="5.08"/>
+<instance part="BAT001" gate="G$1" x="22.86" y="25.4"/>
+<instance part="BAT003" gate="G$1" x="22.86" y="-15.24"/>
 <instance part="BAT002" gate="G$1" x="22.86" y="5.08"/>
+<instance part="VSS8" gate="G$1" x="41.91" y="-24.13"/>
 </instances>
 <busses>
 </busses>
 <nets>
+<net name="VSS" class="0">
+<segment>
+<wire x1="41.91" y1="30.48" x2="41.91" y2="2.54" width="0.1524" layer="91"/>
+<pinref part="VSS8" gate="G$1" pin="VSS"/>
+<pinref part="BAT001" gate="G$1" pin="4"/>
+<wire x1="41.91" y1="2.54" x2="41.91" y2="-10.16" width="0.1524" layer="91"/>
+<wire x1="41.91" y1="-10.16" x2="41.91" y2="-21.59" width="0.1524" layer="91"/>
+<wire x1="27.94" y1="30.48" x2="41.91" y2="30.48" width="0.1524" layer="91"/>
+<pinref part="BAT003" gate="G$1" pin="4"/>
+<wire x1="27.94" y1="-10.16" x2="41.91" y2="-10.16" width="0.1524" layer="91"/>
+<junction x="41.91" y="-10.16"/>
+<pinref part="BAT002" gate="G$1" pin="1"/>
+<wire x1="27.94" y1="2.54" x2="41.91" y2="2.54" width="0.1524" layer="91"/>
+<junction x="41.91" y="2.54"/>
+</segment>
+</net>
+<net name="SENSE1" class="0">
+<segment>
+<pinref part="BAT001" gate="G$1" pin="1"/>
+<wire x1="27.94" y1="22.86" x2="30.48" y2="22.86" width="0.1524" layer="91"/>
+<label x="30.48" y="22.86" size="1.778" layer="95"/>
+</segment>
+</net>
+<net name="SENSE2" class="0">
+<segment>
+<pinref part="BAT002" gate="G$1" pin="4"/>
+<wire x1="27.94" y1="10.16" x2="30.48" y2="10.16" width="0.1524" layer="91"/>
+<label x="30.48" y="10.16" size="1.778" layer="95"/>
+</segment>
+</net>
+<net name="SENSE3" class="0">
+<segment>
+<pinref part="BAT003" gate="G$1" pin="1"/>
+<wire x1="27.94" y1="-17.78" x2="30.48" y2="-17.78" width="0.1524" layer="91"/>
+<label x="30.48" y="-17.78" size="1.778" layer="95"/>
+</segment>
+</net>
 </nets>
 </sheet>
@@
 <instance part="VSS3" gate="G$1" x="12.7" y="-22.86"/>
 <instance part="VSS4" gate="G$1" x="40.64" y="-22.86"/>
-<instance part="SUPPLY1" gate="G$1" x="15.24" y="-15.24" rot="R270"/>
-<instance part="SUPPLY2" gate="G$1" x="43.18" y="-15.24" rot="R270"/>
-<instance part="SUPPLY3" gate="G$1" x="43.18" y="5.08" rot="R270"/>
-<instance part="SUPPLY4" gate="G$1" x="15.24" y="5.08" rot="R270"/>
+<instance part="U$14" gate="G$1" x="12.7" y="5.08" rot="R270"/>
+<instance part="U$15" gate="G$1" x="13.97" y="-15.24" rot="R270"/>
+<instance part="U$16" gate="G$1" x="41.91" y="-15.24" rot="R270"/>
+<instance part="U$17" gate="G$1" x="41.91" y="5.08" rot="R270"/>
 </instances>
 <busses>
@@
 </segment>
 </net>
-<net name="+6V" class="0">
-<segment>
-<pinref part="SUPPLY1" gate="G$1" pin="+7V"/>
-<pinref part="JP3" gate="G$1" pin="2"/>
-<wire x1="12.7" y1="-15.24" x2="10.16" y2="-15.24" width="0.1524" layer="91"/>
-</segment>
-<segment>
-<pinref part="SUPPLY4" gate="G$1" pin="+7V"/>
-<pinref part="JP1" gate="G$1" pin="2"/>
-<wire x1="12.7" y1="5.08" x2="10.16" y2="5.08" width="0.1524" layer="91"/>
-</segment>
-<segment>
-<pinref part="SUPPLY3" gate="G$1" pin="+7V"/>
-<pinref part="JP2" gate="G$1" pin="2"/>
-<wire x1="40.64" y1="5.08" x2="38.1" y2="5.08" width="0.1524" layer="91"/>
-</segment>
-<segment>
-<pinref part="SUPPLY2" gate="G$1" pin="+7V"/>
-<pinref part="JP4" gate="G$1" pin="2"/>
-<wire x1="40.64" y1="-15.24" x2="38.1" y2="-15.24" width="0.1524" layer="91"/>
-</segment>
-</net>
 <net name="SERVO01" class="0">
 <segment>
@@
 </segment>
 </net>
+<net name="P$1" class="0">
+<segment>
+<pinref part="JP3" gate="G$1" pin="2"/>
+<pinref part="U$15" gate="G$1" pin="P$1"/>
+<wire x1="10.16" y1="-15.24" x2="13.97" y2="-15.24" width="0.1524" layer="91"/>
+</segment>
+<segment>
+<pinref part="JP1" gate="G$1" pin="2"/>
+<pinref part="U$14" gate="G$1" pin="P$1"/>
+<wire x1="10.16" y1="5.08" x2="12.7" y2="5.08" width="0.1524" layer="91"/>
+</segment>
+<segment>
+<pinref part="JP2" gate="G$1" pin="2"/>
+<pinref part="U$17" gate="G$1" pin="P$1"/>
+<wire x1="38.1" y1="5.08" x2="41.91" y2="5.08" width="0.1524" layer="91"/>
+</segment>
+<segment>
+<pinref part="JP4" gate="G$1" pin="2"/>
+<pinref part="U$16" gate="G$1" pin="P$1"/>
+<wire x1="38.1" y1="-15.24" x2="41.91" y2="-15.24" width="0.1524" layer="91"/>
+</segment>
+</net>

Commit message: Mejoras en placa de Actuadores y otros
Connections:
- net +24V renamed +22V
- removed net P$1: JP1.2, JP2.2, JP3.2, JP4.2, U$1.PIN19
- new net +11V1: U$1.PIN19, U$12.ROJO
- new net +6V: JP1.2, JP2.2, JP3.2, JP4.2, U$1.PIN20
- net +12V: no longer U$12.ROJO
- net +3V3: now also U$1.PIN22; no longer U$1.PIN21
- net +5V: now also U$1.PIN21; no longer U$1.PIN20
Other:
- note removed: "+6V"

Commit message: Monitor Baterias LiPO
Connections:
- removed net +12V: U$1.PIN18
- removed net +3V3: U$1.PIN22
- removed net +5V: U$1.PIN21
Changed lines of the file:
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@@
 <part name="U$14" library="aasanchez" deviceset="11V1" device=""/>
 <part name="U$15" library="aasanchez" deviceset="+6V" device=""/>
-<part name="P+1" library="supply1" deviceset="+5V" device=""/>
-<part name="+3V1" library="supply1" deviceset="+3V3" device=""/>
-<part name="P+2" library="supply1" deviceset="+12V" device=""/>
 <part name="U$16" library="aasanchez" deviceset="+22V2" device=""/>
 <part name="U$17" library="aasanchez" deviceset="11V1" device=""/>
@@
 <instance part="U$14" gate="G$1" x="96.52" y="30.48" rot="R180"/>
 <instance part="U$15" gate="G$1" x="104.14" y="33.02" rot="R180"/>
-<instance part="P+1" gate="1" x="111.76" y="30.48" rot="R180"/>
-<instance part="+3V1" gate="G$1" x="119.38" y="30.48" rot="R180"/>
-<instance part="P+2" gate="1" x="88.9" y="30.48" rot="R180"/>
 </instances>
 <busses>
@@
 </segment>
 </net>
-<net name="+12V" class="0">
-<segment>
-<pinref part="U$1" gate="G$1" pin="PIN18"/>
-<pinref part="P+2" gate="1" pin="+12V"/>
-<wire x1="73.66" y1="40.64" x2="88.9" y2="40.64" width="0.1524" layer="91"/>
-<wire x1="88.9" y1="40.64" x2="88.9" y2="33.02" width="0.1524" layer="91"/>
-</segment>
-</net>
 <net name="+11V1" class="0">
 <segment>
@@
 </segment>
 </net>
-<net name="+5V" class="0">
-<segment>
-<pinref part="U$1" gate="G$1" pin="PIN21"/>
-<pinref part="P+1" gate="1" pin="+5V"/>
-<wire x1="73.66" y1="48.26" x2="111.76" y2="48.26" width="0.1524" layer="91"/>
-<wire x1="111.76" y1="48.26" x2="111.76" y2="33.02" width="0.1524" layer="91"/>
-</segment>
-</net>
-<net name="+3V3" class="0">
-<segment>
-<pinref part="U$1" gate="G$1" pin="PIN22"/>
-<pinref part="+3V1" gate="G$1" pin="+3V3"/>
-<wire x1="73.66" y1="50.8" x2="119.38" y2="50.8" width="0.1524" layer="91"/>
-<wire x1="119.38" y1="50.8" x2="119.38" y2="33.02" width="0.1524" layer="91"/>
-</segment>
-</net>
