File: Eagle/TG-Final/control.brd (EAGLE design)
At the start: 172.7 x 172.7 mm, 3 parts

Commit message: Listo Placas
Parts:
- removed JP1: (no value), SparkFun:1X06_LONGPADS
- removed U$2: UK1122, aasanchez:UK1122
- added U$3: BLUESMIRF, aasanchez:BLUESMIRF
- added UK1122: UK1122, aasanchez:UK1122
Connections:
- removed net N$3: U$2.MOT2R
- removed net N$4: U$2.MOT2A
- removed net N$5: U$2.MOT1R
- removed net N$6: U$2.MOT1A
- new net M1-A: U$1.PIN05, UK1122.IN1
- new net M1-B: U$1.PIN03, UK1122.EN2
- new net M1-BLACK: U$1.PIN28, UK1122.MOT1A
- new net M1-RED: U$1.PIN29, UK1122.MOT1R
- new net M2-A: U$1.PIN02, UK1122.IN3
- new net M2-B: U$1.PIN00, UK1122.IN4
- new net M2-BLACK: U$1.PIN31, UK1122.MOT2A
- new net M2-RED: U$1.PIN30, UK1122.MOT2R
- new net PWM1: U$1.PIN04, UK1122.ENA
- new net PWM2: U$1.PIN01, UK1122.ENB
- new net RX: U$1.PIN06, U$3.TX-O
- new net TX: U$1.PIN07, U$3.RX-I
- net +12V: now also U$1.PIN18, UK1122.+; no longer U$2.+
- net VDD: now also U$1.PIN21, U$3.VDD, UK1122.+5; no longer U$2.+5
- net VSS: now also U$1.PIN16, U$3.VSS, UK1122.-, UK1122.GND; no longer U$2.-, U$2.CSA, U$2.CSB, U$2.GND
Routing:
- net +12V: track 0.00 -> 221.6 mm, vias 0 -> 2
- net VDD: track 0.00 -> 169.5 mm, vias 0 -> 4
- net VSS: track 0.00 -> 139.0 mm
- net M2-B: track 0.00 -> 119.6 mm
- net PWM2: track 0.00 -> 112.2 mm
- net M2-A: track 0.00 -> 108.7 mm
- net M1-BLACK: track 0.00 -> 107.3 mm
- net M1-B: track 0.00 -> 104.0 mm
- net PWM1: track 0.00 -> 100.4 mm
- net M2-BLACK: track 0.00 -> 98.6 mm
- net M1-A: track 0.00 -> 96.1 mm
- net M2-RED: track 0.00 -> 94.3 mm
- net RX: track 0.00 -> 92.6 mm
- net M1-RED: track 0.00 -> 91.7 mm
- net TX: track 0.00 -> 81.4 mm
- added copper zone on layer 16, net VSS
