File: Eagle/TG-Final/control.sch (EAGLE design)
At the start: 3 parts

Commit message: Listo Placas
Parts:
- removed JP1: (no value), SparkFun:M06LONGPADS
- added U$3: BLUESMIRF, aasanchez:BLUESMIRF
- renumbered U$2 to UK1122
Connections:
- removed net N$3: UK1122.MOT2R
- removed net N$4: UK1122.MOT2A
- removed net N$5: UK1122.MOT1R
- removed net N$6: UK1122.MOT1A
- new net M1-A: U$1.PIN05, UK1122.IN1
- new net M1-B: U$1.PIN03, UK1122.IN2
- new net M1-BLACK: U$1.PIN28, UK1122.MOT1A
- new net M1-RED: U$1.PIN29, UK1122.MOT1R
- new net M2-A: U$1.PIN02, UK1122.IN3
- new net M2-B: U$1.PIN00, UK1122.IN4
- new net M2-BLACK: U$1.PIN31, UK1122.MOT2A
- new net M2-RED: U$1.PIN30, UK1122.MOT2R
- new net PWM1: U$1.PIN04, UK1122.ENA
- new net PWM2: U$1.PIN01, UK1122.ENB
- new net RX: U$1.PIN06, U$3.TX-O
- new net TX: U$1.PIN07, U$3.RX-I
- net +12V: now also U$1.+12V
- net VDD: now also U$1.+5V, U$3.VDD
- net VSS: now also U$1.VSS, U$3.VSS; no longer UK1122.CSA, UK1122.CSB
