File: Eagle/TG-Final/nivel0-2.brd (EAGLE design)
At the start: 172.7 x 172.7 mm, 21 parts

Commit message: Actualizaciones Varias
Connections:
- net SENSE1 renamed V-BAT1
- removed net SENSE2: BAT002.4, U$1.PIN13
- removed net SENSE3: BAT003.1, U$1.PIN14
- new net GND: U$1.PIN23, U$12.P$1
- new net GND-BAT1: BAT001.4, U$1.PIN14
- new net GND-BAT2: BAT002.1, U$1.PIN10
- new net GND-BAT3: BAT003.4, U$1.PIN12
- new net V-BAT2: BAT002.4, U$1.PIN11
- new net V-BAT3: BAT003.1, U$1.PIN13
- net VSS: no longer BAT001.4, BAT002.1, BAT003.4, U$12.P$1
Routing:
- net SENSE2: track 280.2 -> 0.00 mm, vias 4 -> 0
- net V-BAT1: track 156.1 -> 0.00 mm, vias 2 -> 0
- net VSS: track 510.6 -> 370.2 mm
- net SENSE3: track 139.0 -> 0.00 mm, vias 2 -> 0
