File: Eagle/TG-Final/brain.brd (EAGLE design)
At the start: 172.7 x 172.7 mm, 5 parts

Commit message: Placa de Control Motores y Comunicación
Parts:
- removed U$5: UK1122, aasanchez:UK1122
- moved U$8 83.9 mm to (-127.0, 80.0), turned to 0 degrees
- moved U$6 72.5 mm to (-95.2, 50.8), flipped to the bottom, turned to 90 degrees
- moved U$7 56.4 mm to (-141.0, 100.3), turned to 180 degrees
Connections:
- removed net +: U$5.+
- removed net +5: U$5.+5
- removed net -: U$5.-
- removed net LV: U$8.P$3
- new net N$1: U$1.PIN15
- new net N$2: U$1.PIN14
- new net N$3: U$1.PIN13
- net +3V3: now also U$8.P$3
- net GND: no longer U$5.GND, U$8.P$4
- net VSS: now also U$8.P$4
Changed lines of the file:
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@@
 <board>
 <plain>
+<wire x1="0" y1="0" x2="160" y2="0" width="0" layer="20"/>
+<wire x1="160" y1="0" x2="160" y2="100" width="0" layer="20"/>
+<wire x1="160" y1="100" x2="0" y2="100" width="0" layer="20"/>
+<wire x1="0" y1="100" x2="0" y2="0" width="0" layer="20"/>
 </plain>
 <attributes>
@@
 <elements>
 <element name="U$1" library="aasanchez" package="BASE" value="BASE" x="-100.33" y="87.63"/>
-<element name="U$6" library="adafruit" package="ARDUINO-NOHOLE" value="ARDUINO-NOHOLE" x="-81.28" y="121.92" rot="R270"/>
-<element name="U$5" library="aasanchez" package="UK1122" value="UK1122" x="-95.25" y="55.88" rot="R90"/>
-<element name="U$7" library="aasanchez" package="IMU3000-COMBO" value="IMU3000COMBO" x="-95.25" y="133.35" rot="R90"/>
-<element name="U$8" library="aasanchez" package="LEVEL-CONVERTER" value="LOGIC-LEVEL-CONVERTER" x="-82.55" y="151.13" rot="R180"/>
+<element name="U$6" library="adafruit" package="ARDUINO-NOHOLE" value="ARDUINO-NOHOLE" x="-95.25" y="50.8" rot="MR90"/>
+<element name="U$7" library="aasanchez" package="IMU3000-COMBO" value="IMU3000COMBO" x="-140.97" y="100.33" rot="R180"/>
+<element name="U$8" library="aasanchez" package="LEVEL-CONVERTER" value="LOGIC-LEVEL-CONVERTER" x="-127" y="80.01"/>
 </elements>
 <signals>
 <signal name="GND">
 <contactref element="U$6" pad="GND"/>
-<contactref element="U$5" pad="GND"/>
-<contactref element="U$8" pad="P$4"/>
-<wire x1="-30.48" y1="95.504" x2="-74.93" y2="82.55" width="0" layer="19" extent="1-1"/>
-<wire x1="-81.28" y1="144.78" x2="-30.48" y2="95.504" width="0" layer="19" extent="1-1"/>
 </signal>
 <signal name="VIN">
@@
 <signal name="3V">
 <contactref element="U$6" pad="3V"/>
-</signal>
-<signal name="+5">
-<contactref element="U$5" pad="+5"/>
-</signal>
-<signal name="-">
-<contactref element="U$5" pad="-"/>
-</signal>
-<signal name="+">
-<contactref element="U$5" pad="+" route="any"/>
-</signal>
-<signal name="LV">
-<contactref element="U$8" pad="P$3"/>
 </signal>
 <signal name="HV">
@@
 <contactref element="U$1" pad="PIN16"/>
 <contactref element="U$7" pad="VSS"/>
-<wire x1="-104.14" y1="134.62" x2="-109.22" y2="11.43" width="0" layer="19" extent="1-1"/>
+<contactref element="U$8" pad="P$4"/>
+<wire x1="-128.27" y1="86.36" x2="-109.22" y2="11.43" width="0" layer="19" extent="1-1"/>
+<wire x1="-142.24" y1="91.44" x2="-128.27" y2="86.36" width="0" layer="19" extent="1-1"/>
 </signal>
 <signal name="+22V">
@@
 <contactref element="U$1" pad="PIN22"/>
 <contactref element="U$7" pad="3V3"/>
-<wire x1="-101.6" y1="134.62" x2="-93.98" y2="11.43" width="0" layer="19" extent="1-1"/>
+<contactref element="U$8" pad="P$3"/>
+<wire x1="-142.24" y1="93.98" x2="-93.98" y2="11.43" width="0" layer="19" extent="1-1"/>
+<wire x1="-128.27" y1="88.9" x2="-142.24" y2="93.98" width="0" layer="19" extent="1-1"/>
+</signal>
+<signal name="N$1">
+<contactref element="U$1" pad="PIN15"/>
+</signal>
+<signal name="N$2">
+<contactref element="U$1" pad="PIN14"/>
+</signal>
+<signal name="N$3">
+<contactref element="U$1" pad="PIN13"/>
 </signal>
 </signals>

Commit message: Listo Placas
Parts:
- added U$3: (no value), OSHW:OSHW_FILLX1000_NOTEXT
- U$6: value ARDUINO-NOHOLE -> ARDUINOUNO; device adafruit:ARDUINO-NOHOLE -> adafruit:ARDUINO
- moved U$7 39.6 mm to (-170.2, 73.7), turned to 0 degrees
- moved U$8 15.7 mm to (-123.2, 95.2), flipped to the bottom, turned to 180 degrees
- moved U$6 8.98 mm to (-88.9, 57.1)
Connections:
- removed net : U$8.P$9
- removed net +11V1: U$1.PIN19
- removed net +12V: U$1.PIN18
- removed net +22V: U$1.PIN17
- removed net +6V: U$1.PIN20
- removed net 5V: U$6.5V
- removed net GND1: U$6.GND1
- removed net GND2: U$6.GND2
- removed net HV: U$8.P$10
- removed net N$3: U$1.PIN13
- new net M1-A: U$1.PIN05, U$6.D13
- new net M1-B: U$1.PIN03, U$6.D12
- new net M2-A: U$1.PIN02, U$6.D8
- new net M2-B: U$1.PIN00, U$6.D7
- new net PWM1: U$1.PIN04, U$6.D11
- new net PWM2: U$1.PIN01, U$6.D9
- new net RX: U$1.PIN06, U$6.D0
- new net SCL: U$6.A5, U$8.P$12
- new net SDA: U$6.A4, U$8.P$7
- new net SERVO1: U$1.PIN24, U$6.D10
- new net SERVO2: U$1.PIN27, U$6.D3
- new net SERVO3: U$1.PIN26, U$6.D5
- new net SERVO4: U$1.PIN25, U$6.D6
- new net TX: U$1.PIN07, U$6.D1
- net N$1: now also U$7.SCL, U$8.P$1; no longer U$1.PIN15
- net N$2: now also U$7.SDA, U$8.P$6; no longer U$1.PIN14
- net VDD: now also U$6.5V, U$8.P$10
- net VSS: now also U$6.GND1, U$6.GND2, U$8.P$9
Routing:
- net VSS: track 0.00 -> 259.9 mm, vias 0 -> 2
- net +3V3: track 0.00 -> 162.2 mm
- net M1-A: track 0.00 -> 141.4 mm
- net TX: track 0.00 -> 136.3 mm
- net PWM1: track 0.00 -> 133.8 mm, vias 0 -> 2
- net M1-B: track 0.00 -> 133.8 mm
- net VDD: track 0.00 -> 132.8 mm
- net M2-A: track 0.00 -> 121.1 mm, vias 0 -> 2
- net PWM2: track 0.00 -> 121.1 mm
- net RX: track 0.00 -> 119.3 mm
- net M2-B: track 0.00 -> 111.7 mm
- net N$1: track 0.00 -> 76.5 mm
- net SDA: track 0.00 -> 58.4 mm
- net SCL: track 0.00 -> 56.9 mm
- net N$2: track 0.00 -> 51.1 mm
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- added copper zone on layer 16, net N$3
- added copper zone on layer 16, net N$4
Other:
- board text added: "Alexis A. Sánchez"
- board text added: "BP"
- board text added: "Balanced Pendulum"
- board text added: "LV"

Commit message: Actualizaciones Varias
Connections:
- net 3V renamed N$5

Commit message: Nuevo diseño
Connections:
- net SERVO1: no longer U$1.PIN24
- net SERVO2: no longer U$1.PIN27
- net SERVO3: no longer U$1.PIN26
- net SERVO4: no longer U$1.PIN25
Routing:
- net SERVO1: track 27.6 -> 18.7 mm
- net SERVO4: track 36.6 -> 29.0 mm
- net SERVO3: track 36.6 -> 30.3 mm
- net SERVO2: track 39.2 -> 34.1 mm
Changed lines of the file:
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@@
 <signal name="SERVO4">
 <contactref element="U$6" pad="D6"/>
-<contactref element="U$1" pad="PIN25"/>
-<wire x1="-24.13" y1="81.28" x2="-31.75" y2="81.28" width="0.6096" layer="16"/>
 <wire x1="-31.75" y1="81.28" x2="-33.02" y2="82.55" width="0.6096" layer="16"/>
 <wire x1="-33.02" y1="82.55" x2="-33.02" y2="104.14" width="0.6096" layer="16"/>
@@
 <signal name="SERVO2">
 <contactref element="U$6" pad="D3"/>
-<contactref element="U$1" pad="PIN27"/>
-<wire x1="-24.13" y1="86.36" x2="-29.21" y2="86.36" width="0.6096" layer="16"/>
 <wire x1="-29.21" y1="86.36" x2="-30.48" y2="87.63" width="0.6096" layer="16"/>
 <wire x1="-30.48" y1="87.63" x2="-30.48" y2="111.76" width="0.6096" layer="16"/>
@@
 <signal name="SERVO3">
 <contactref element="U$6" pad="D5"/>
-<contactref element="U$1" pad="PIN26"/>
-<wire x1="-24.13" y1="83.82" x2="-30.48" y2="83.82" width="0.6096" layer="16"/>
 <wire x1="-30.48" y1="83.82" x2="-31.75" y2="85.09" width="0.6096" layer="16"/>
 <wire x1="-31.75" y1="85.09" x2="-31.75" y2="106.68" width="0.6096" layer="16"/>
@@
 <signal name="SERVO1">
 <contactref element="U$6" pad="D10"/>
-<contactref element="U$1" pad="PIN24"/>
 <wire x1="-38.1" y1="93.726" x2="-35.306" y2="93.726" width="0.6096" layer="16"/>
 <wire x1="-35.306" y1="93.726" x2="-34.29" y2="92.71" width="0.6096" layer="16"/>
 <wire x1="-34.29" y1="92.71" x2="-34.29" y2="80.01" width="0.6096" layer="16"/>
 <wire x1="-34.29" y1="80.01" x2="-33.02" y2="78.74" width="0.6096" layer="16"/>
-<wire x1="-33.02" y1="78.74" x2="-24.13" y2="78.74" width="0.6096" layer="16"/>
 </signal>
 <signal name="N$3">
