File: Eagle/TG-Final/arduino.sch (EAGLE design)
At the start: 4 parts

Commit message: Nuevo diseño
Parts:
- U$1: value BASE -> BASEFINAL; device aasanchez:BASE -> aasanchez:BASEFINAL
- U$6: value ARDUINOUNO -> ARDUINO-NOHOLE; device adafruit:ARDUINOUNO -> adafruit:ARDUINO-NOHOLE
Connections:
- removed net M1-A: U$1.PIN05, U$6.D13
- removed net M1-B: U$1.PIN03, U$6.D12
- removed net M2-A: U$1.PIN02, U$6.D8
- removed net M2-B: U$1.PIN00, U$6.D7
- removed net N$5: U$6.3V
- removed net PWM1: U$1.PIN04, U$6.PWM-D11
- removed net PWM2: U$1.PIN01, U$6.PWM-D9
- removed net RX: U$1.PIN06, U$6.RX-D0
- removed net SCL: U$6.A5-SCL, U$8.TXO-1
- removed net SDA: U$6.A4-SDA, U$8.TXO-2
- removed net SERVO1: U$6.PWM-D10
- removed net SERVO2: U$6.PWM-D3
- removed net SERVO3: U$6.PWM-D5
- removed net SERVO4: U$6.PWM-D6
- removed net TX: U$1.PIN07, U$6.TX-D1
- removed net VDD: U$1.+5V, U$6.5V, U$8.HV
- removed net VSS: U$1.VSS, U$6.GND1, U$6.GND2, U$7.GND, U$8.@GND, U$8.GND
- new net PIN09: U$1.PIN09, U$6./RESET
- new net PIN10: U$1.PIN10, U$6.5V, U$8.HV
- new net PIN11: U$1.PIN11, U$6.GND1, U$6.GND2, U$7.GND, U$8.@GND, U$8.GND
- new net PIN12: U$1.PIN12, U$6.A0
- new net PIN13: U$1.PIN13, U$6.A1
- new net PIN14: U$1.PIN14, U$6.A2
- new net PIN15: U$1.PIN15, U$6.A3
- new net PIN16: U$1.PIN16, U$6.RX-D0
- new net PIN17: U$1.PIN17, U$6.TX-D1
- new net PIN18: U$1.PIN18, U$6.D2
- new net PIN19: U$1.PIN19, U$6.PWM-D3
- new net PIN20: U$1.PIN20, U$6.D4
- new net PIN21: U$1.PIN21, U$6.PWM-D5
- new net PIN22: U$1.PIN22, U$6.PWM-D6
- new net PIN23: U$1.PIN23, U$6.D7
- new net PIN24: U$1.PIN24, U$6.D8
- new net PIN25: U$1.PIN25, U$6.PWM-D9
- new net PIN26: U$1.PIN26, U$6.PWM-D10
- new net PIN27: U$1.PIN27, U$6.PWM-D11
- new net PIN28: U$1.PIN28, U$6.D12
- new net PIN29: U$1.PIN29, U$6.D13
- new net PIN30: U$1.PIN30, U$6.A4-SDA, U$8.TXO-2
- new net PIN31: U$1.PIN31, U$6.A5-SCL, U$8.TXO-1
- net +3V3: now also U$6.3V; no longer U$1.+3V3

Commit message: Muchos Cambios a 2 dias de la denfesa
Parts:
- added LED1: (no value), SparkFun:LED3MM
- added R1: (no value), SparkFun:RESISTORKIT
- added S1: (no value), switch-omron:10-XX
- added S2: TL39YOSWITCH_2_ESTADOS, aasanchez:TL39YOSWITCH_2_ESTADOS
- U$1: value BASEFINAL -> BASE-FINAL; device aasanchez:BASEFINAL -> aasanchez:BASE-FINAL
Connections:
- removed net PIN09: U$1.PIN09, U$6./RESET
- removed net PIN10: U$1.PIN10, U$6.5V, U$8.HV
- removed net PIN11: U$1.PIN11, U$6.GND1, U$6.GND2, U$7.GND, U$8.@GND, U$8.GND
- removed net PIN12: U$1.PIN12, U$6.A0
- removed net PIN13: U$1.PIN13, U$6.A1
- removed net PIN14: U$1.PIN14, U$6.A2
- removed net PIN15: U$1.PIN15, U$6.A3
- removed net PIN30: U$1.PIN30, U$6.A4-SDA, U$8.TXO-2
- removed net PIN31: U$1.PIN31, U$6.A5-SCL, U$8.TXO-1
- new net 5V: U$1.5V, U$6.5V, U$8.HV
- new net A0: U$1.A0, U$6.A0
- new net A1: U$1.A1, U$6.A1
- new net A2: U$1.A2, U$6.A2
- new net A3: U$1.A3, U$6.A3
- new net A4: U$1.A4, U$6.A4-SDA, U$8.TXO-2
- new net A5: U$1.A5, U$6.A5-SCL, U$8.TXO-1
- new net GND: R1.1, S1.P, U$1.GND, U$6.GND, U$6.GND1, U$6.GND2, U$7.GND, U$8.@GND, U$8.GND
- new net N$4: S2.P, U$1.VIN
- new net N$5: LED1.C, R1.2
- new net RST: S1.S1, U$1.RST, U$6./RESET
- new net VIN: S2.O, U$6.VIN
- net PIN16: now also U$1.D0; no longer U$1.PIN16
- net PIN17: now also U$1.D1; no longer U$1.PIN17
- net PIN18: now also U$1.D2; no longer U$1.PIN18
- net PIN19: now also U$1.D3; no longer U$1.PIN19
- net PIN20: now also U$1.D4; no longer U$1.PIN20
- net PIN21: now also U$1.D5; no longer U$1.PIN21
- net PIN22: now also U$1.D6; no longer U$1.PIN22
- net PIN23: now also U$1.D7; no longer U$1.PIN23
- net PIN24: now also U$1.D8; no longer U$1.PIN24
- net PIN25: now also U$1.D9; no longer U$1.PIN25
- net PIN26: now also U$1.D10; no longer U$1.PIN26
- net PIN27: now also LED1.A, U$1.D11; no longer U$1.PIN27
- net PIN28: now also U$1.D12; no longer U$1.PIN28
- net PIN29: now also U$1.D13; no longer U$1.PIN29
