File: Eagle/TG-Final/uk1122.sch (EAGLE design)
At the start: 2 parts

Commit message: Muchos Cambios a 2 dias de la denfesa
Parts:
- U$1: value BASEFINAL -> BASE-FINAL; device aasanchez:BASEFINAL -> aasanchez:BASE-FINAL
Connections:
- net N$3 renamed MOT2R
- net N$4 renamed MOT2A
- removed net N$12: U$1.PIN23, U$2.IN4
- removed net N$14: U$1.PIN14, U$2.CSB
- new net CSB: U$1.A2, U$2.CSB
- new net IN4: U$1.D7, U$2.IN4
- new net N$21: U$1.GND, U$2.-, U$2.VDD
- net N$10: now also U$1.A3; no longer U$1.PIN15
- net N$11: now also U$1.D8; no longer U$1.PIN24
- net N$13: now also U$1.D6; no longer U$1.PIN22
- net N$5: now also U$1.5V; no longer U$1.PIN10
- net N$6: now also U$1.11V1, U$2.+; no longer U$1.PIN11, U$2.VDD
- net N$7: now also U$1.D13; no longer U$1.PIN29
- net N$8: now also U$1.D12; no longer U$1.PIN28
- net N$9: now also U$1.D5; no longer U$1.PIN21
Changed lines of the file:
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@@
 </classes>
 <parts>
-<part name="U$1" library="aasanchez" deviceset="BASE" device="FINAL"/>
+<part name="U$1" library="aasanchez" deviceset="BASE-FINAL" device=""/>
 <part name="U$2" library="aasanchez" deviceset="UK1122" device="FINO"/>
 </parts>
@@
 </segment>
 </net>
-<net name="N$3" class="0">
+<net name="MOT2R" class="0">
 <segment>
 <pinref part="U$2" gate="G$1" pin="MOT2R"/>
-<wire x1="99.06" y1="-7.62" x2="99.06" y2="-17.78" width="0.1524" layer="91"/>
-<wire x1="99.06" y1="-17.78" x2="-10.16" y2="-17.78" width="0.1524" layer="91"/>
-<wire x1="-10.16" y1="-17.78" x2="-10.16" y2="35.56" width="0.1524" layer="91"/>
+<wire x1="99.06" y1="-7.62" x2="99.06" y2="-15.24" width="0.1524" layer="91"/>
+<label x="109.22" y="-15.24" size="1.778" layer="95" rot="R180"/>
+</segment>
+<segment>
 <pinref part="U$1" gate="G$1" pin="PIN02"/>
-<wire x1="-10.16" y1="35.56" x2="-5.08" y2="35.56" width="0.1524" layer="91"/>
-</segment>
-</net>
-<net name="N$4" class="0">
-<segment>
-<pinref part="U$2" gate="G$1" pin="MOT2A"/>
-<wire x1="96.52" y1="-7.62" x2="96.52" y2="-15.24" width="0.1524" layer="91"/>
-<wire x1="96.52" y1="-15.24" x2="-7.62" y2="-15.24" width="0.1524" layer="91"/>
-<wire x1="-7.62" y1="-15.24" x2="-7.62" y2="33.02" width="0.1524" layer="91"/>
-<pinref part="U$1" gate="G$1" pin="PIN03"/>
-<wire x1="-7.62" y1="33.02" x2="-5.08" y2="33.02" width="0.1524" layer="91"/>
+<wire x1="-7.62" y1="35.56" x2="-5.08" y2="35.56" width="0.1524" layer="91"/>
+<label x="-20.32" y="35.56" size="1.778" layer="95"/>
 </segment>
 </net>
@@
 <wire x1="68.58" y1="25.4" x2="68.58" y2="48.26" width="0.1524" layer="91"/>
 <wire x1="68.58" y1="48.26" x2="-17.78" y2="48.26" width="0.1524" layer="91"/>
-<wire x1="-17.78" y1="48.26" x2="-17.78" y2="15.24" width="0.1524" layer="91"/>
-<pinref part="U$1" gate="G$1" pin="PIN10"/>
-<wire x1="-17.78" y1="15.24" x2="-5.08" y2="15.24" width="0.1524" layer="91"/>
-</segment>
-</net>
-<net name="N$6" class="0">
-<segment>
-<pinref part="U$2" gate="G$1" pin="VDD"/>
-<wire x1="71.12" y1="22.86" x2="66.04" y2="22.86" width="0.1524" layer="91"/>
-<wire x1="66.04" y1="22.86" x2="66.04" y2="50.8" width="0.1524" layer="91"/>
-<wire x1="66.04" y1="50.8" x2="-20.32" y2="50.8" width="0.1524" layer="91"/>
-<wire x1="-20.32" y1="50.8" x2="-20.32" y2="12.7" width="0.1524" layer="91"/>
-<pinref part="U$1" gate="G$1" pin="PIN11"/>
-<wire x1="-20.32" y1="12.7" x2="-5.08" y2="12.7" width="0.1524" layer="91"/>
+<wire x1="-17.78" y1="48.26" x2="-17.78" y2="17.78" width="0.1524" layer="91"/>
+<pinref part="U$1" gate="G$1" pin="5V"/>
+<wire x1="-17.78" y1="17.78" x2="-5.08" y2="17.78" width="0.1524" layer="91"/>
 </segment>
 </net>
@@
 <wire x1="71.12" y1="20.32" x2="63.5" y2="20.32" width="0.1524" layer="91"/>
 <wire x1="63.5" y1="20.32" x2="63.5" y2="35.56" width="0.1524" layer="91"/>
-<pinref part="U$1" gate="G$1" pin="PIN29"/>
+<pinref part="U$1" gate="G$1" pin="D13"/>
 <wire x1="63.5" y1="35.56" x2="40.64" y2="35.56" width="0.1524" layer="91"/>
 </segment>
@@
 <wire x1="71.12" y1="15.24" x2="60.96" y2="15.24" width="0.1524" layer="91"/>
 <wire x1="60.96" y1="15.24" x2="60.96" y2="33.02" width="0.1524" layer="91"/>
-<pinref part="U$1" gate="G$1" pin="PIN28"/>
+<pinref part="U$1" gate="G$1" pin="D12"/>
 <wire x1="60.96" y1="33.02" x2="40.64" y2="33.02" width="0.1524" layer="91"/>
 </segment>
@@
 <wire x1="71.12" y1="17.78" x2="53.34" y2="17.78" width="0.1524" layer="91"/>
 <wire x1="53.34" y1="17.78" x2="53.34" y2="15.24" width="0.1524" layer="91"/>
-<pinref part="U$1" gate="G$1" pin="PIN21"/>
+<pinref part="U$1" gate="G$1" pin="D5"/>
 <wire x1="53.34" y1="15.24" x2="40.64" y2="15.24" width="0.1524" layer="91"/>
 </segment>
@@
 <segment>
 <pinref part="U$2" gate="G$1" pin="CSA"/>
-<wire x1="71.12" y1="12.7" x2="68.58" y2="12.7" width="0.1524" layer="91"/>
-<wire x1="68.58" y1="12.7" x2="68.58" y2="-5.08" width="0.1524" layer="91"/>
-<wire x1="68.58" y1="-5.08" x2="-17.78" y2="-5.08" width="0.1524" layer="91"/>
+<wire x1="71.12" y1="12.7" x2="45.72" y2="12.7" width="0.1524" layer="91"/>
+<wire x1="45.72" y1="12.7" x2="45.72" y2="-5.08" width="0.1524" layer="91"/>
+<wire x1="45.72" y1="-5.08" x2="-17.78" y2="-5.08" width="0.1524" layer="91"/>
 <wire x1="-17.78" y1="-5.08" x2="-17.78" y2="2.54" width="0.1524" layer="91"/>
-<pinref part="U$1" gate="G$1" pin="PIN15"/>
+<pinref part="U$1" gate="G$1" pin="A3"/>
 <wire x1="-17.78" y1="2.54" x2="-5.08" y2="2.54" width="0.1524" layer="91"/>
 </segment>
@@
 <wire x1="71.12" y1="10.16" x2="58.42" y2="10.16" width="0.1524" layer="91"/>
 <wire x1="58.42" y1="10.16" x2="58.42" y2="22.86" width="0.1524" layer="91"/>
-<pinref part="U$1" gate="G$1" pin="PIN24"/>
+<pinref part="U$1" gate="G$1" pin="D8"/>
 <wire x1="58.42" y1="22.86" x2="40.64" y2="22.86" width="0.1524" layer="91"/>
 </segment>
 </net>
-<net name="N$12" class="0">
+<net name="IN4" class="0">
 <segment>
 <pinref part="U$2" gate="G$1" pin="IN4"/>
-<wire x1="71.12" y1="5.08" x2="55.88" y2="5.08" width="0.1524" layer="91"/>
-<wire x1="55.88" y1="5.08" x2="55.88" y2="20.32" width="0.1524" layer="91"/>
-<pinref part="U$1" gate="G$1" pin="PIN23"/>
-<wire x1="55.88" y1="20.32" x2="40.64" y2="20.32" width="0.1524" layer="91"/>
+<wire x1="71.12" y1="5.08" x2="68.58" y2="5.08" width="0.1524" layer="91"/>
+<label x="63.5" y="5.08" size="1.778" layer="95"/>
+</segment>
+<segment>
+<pinref part="U$1" gate="G$1" pin="D7"/>
+<wire x1="43.18" y1="20.32" x2="40.64" y2="20.32" width="0.1524" layer="91"/>
+<label x="43.18" y="20.32" size="1.778" layer="95"/>
 </segment>
 </net>
@@
 <pinref part="U$2" gate="G$1" pin="ENB"/>
 <wire x1="71.12" y1="7.62" x2="50.8" y2="7.62" width="0.1524" layer="91"/>
-<pinref part="U$1" gate="G$1" pin="PIN22"/>
+<pinref part="U$1" gate="G$1" pin="D6"/>
 <wire x1="40.64" y1="17.78" x2="50.8" y2="17.78" width="0.1524" layer="91"/>
 <wire x1="50.8" y1="17.78" x2="50.8" y2="7.62" width="0.1524" layer="91"/>
 </segment>
 </net>
-<net name="N$14" class="0">
+<net name="CSB" class="0">
 <segment>
 <pinref part="U$2" gate="G$1" pin="CSB"/>
-<wire x1="71.12" y1="2.54" x2="66.04" y2="2.54" width="0.1524" layer="91"/>
-<wire x1="66.04" y1="2.54" x2="66.04" y2="-10.16" width="0.1524" layer="91"/>
-<wire x1="66.04" y1="-10.16" x2="-20.32" y2="-10.16" width="0.1524" layer="91"/>
-<wire x1="-20.32" y1="-10.16" x2="-20.32" y2="5.08" width="0.1524" layer="91"/>
-<pinref part="U$1" gate="G$1" pin="PIN14"/>
-<wire x1="-20.32" y1="5.08" x2="-5.08" y2="5.08" width="0.1524" layer="91"/>
+<wire x1="71.12" y1="2.54" x2="68.58" y2="2.54" width="0.1524" layer="91"/>
+<label x="63.5" y="2.54" size="1.778" layer="95"/>
+</segment>
+<segment>
+<pinref part="U$1" gate="G$1" pin="A2"/>
+<wire x1="-7.62" y1="5.08" x2="-5.08" y2="5.08" width="0.1524" layer="91"/>
+<label x="-12.7" y="5.08" size="1.778" layer="95"/>
 </segment>
 </net>
+<net name="N$21" class="0">
+<segment>
+<pinref part="U$2" gate="G$1" pin="-"/>
+<pinref part="U$2" gate="G$1" pin="VDD"/>
+<wire x1="71.12" y1="22.86" x2="66.04" y2="22.86" width="0.1524" layer="91"/>
+<wire x1="66.04" y1="22.86" x2="66.04" y2="50.8" width="0.1524" layer="91"/>
+<wire x1="66.04" y1="50.8" x2="-25.4" y2="50.8" width="0.1524" layer="91"/>
+<wire x1="-25.4" y1="50.8" x2="-25.4" y2="15.24" width="0.1524" layer="91"/>
+<pinref part="U$1" gate="G$1" pin="GND"/>
+<wire x1="-25.4" y1="15.24" x2="-5.08" y2="15.24" width="0.1524" layer="91"/>
+<wire x1="71.12" y1="35.56" x2="71.12" y2="22.86" width="0.1524" layer="91"/>
+</segment>
+</net>
+<net name="N$6" class="0">
+<segment>
+<pinref part="U$1" gate="G$1" pin="11V1"/>
+<wire x1="-5.08" y1="22.86" x2="-12.7" y2="22.86" width="0.1524" layer="91"/>
+<wire x1="-12.7" y1="22.86" x2="-12.7" y2="45.72" width="0.1524" layer="91"/>
+<wire x1="-12.7" y1="45.72" x2="58.42" y2="45.72" width="0.1524" layer="91"/>
+<wire x1="58.42" y1="45.72" x2="58.42" y2="38.1" width="0.1524" layer="91"/>
+<pinref part="U$2" gate="G$1" pin="+"/>
+<wire x1="58.42" y1="38.1" x2="71.12" y2="38.1" width="0.1524" layer="91"/>
+</segment>
+</net>
+<net name="MOT2A" class="0">
+<segment>
+<pinref part="U$2" gate="G$1" pin="MOT2A"/>
+<wire x1="96.52" y1="-7.62" x2="96.52" y2="-15.24" width="0.1524" layer="91"/>
+<label x="96.52" y="-15.24" size="1.778" layer="95" rot="R180"/>
+</segment>
+<segment>
+<pinref part="U$1" gate="G$1" pin="PIN03"/>
+<wire x1="-7.62" y1="33.02" x2="-5.08" y2="33.02" width="0.1524" layer="91"/>
+<label x="-20.32" y="33.02" size="1.778" layer="95"/>
+</segment>
+</net>
